File: soil-moisture-module/soil-moisture-module.sch (KiCad schematic (older format))
At the start: 12 parts, among them J1 MODULE_HEADER, U1 ATTINY24-SS

Commit message: first pass with "active" probes
Parts:
- removed D1: DIODESCH, symbol DIODESCH
- added C5, C6, C7: 100nF, parts:SMD-0402, symbol C
- added D1, D3: DIODE, SMD_Packages:SOT-23, symbol DIODE
- added J2, J3, J4, J5: CONN_02X03, Pin_Headers:Pin_Header_Straight_2x03, symbol CONN_01X06
- added Q1, Q2: nMOS, SMD_Packages:SOT-23-GDS, symbol nMOS
- added R5: 10kR, parts:SMD-0402, symbol R
- added R6: 1MR, parts:SMD-0402, symbol R
- added R7: 1kR, parts:SMD-0402, symbol R
- C1, C2, C4, R1, R3, R4: footprint (none) -> parts:SMD-0402
- C3: value 100nF -> 10pF, DNP; footprint (none) -> parts:SMD-0402
- D2: footprint (none) -> LEDs:LED-0603
- J1: footprint (none) -> parts:MODULE_HEADER_MODULE
- R2: value 0R -> 1kR; footprint (none) -> parts:SMD-0402
- U1: footprint SO14 -> SMD_Packages:SOIC-14_N
Connections:
- net labels added: 3.3V_PROBE_0, 3.3V_PROBE_1, GND0, GND1, LPF0_IN, LPF0_OUT, LPF1_IN, LPF1_OUT, PD0_IN, PD0_OUT, PD1_IN, PD1_OUT, WAVE_AMP_0, WAVE_AMP_1, WAVE_IN_0, WAVE_IN_1, WAVE_OUT
- net labels removed: AREF, LPF, PD, WAVE
- wire segments 67 -> 125
Other:
- note added: "CABLE"
- moved on the sheet: C1, C2, C4, D2, J1, R1, R3, R4, U1

Commit message: tricksy footprints...
Parts:
- removed D1, D3: DIODE, SMD_Packages:SOT-23, symbol DIODE
- added D1, D3: PMBD914,235, SMD_Packages:SOT-23, symbol SCHDPAK
- Q1, Q2: value nMOS -> 2N7002; footprint SMD_Packages:SOT-23-GDS -> SMD_Packages:SOT-23
Connections:
- wire segments 125 -> 127
Changed lines of the file:
@@
 Text Label 3550 6300 0    60   ~ 0
 LPF0_IN
-$Comp
-L DIODE D1
-U 1 1 546C2ECF
-P 8900 2200
-F 0 "D1" H 8900 2300 40  0000 C CNN
-F 1 "DIODE" H 8900 2100 40  0000 C CNN
-F 2 "SMD_Packages:SOT-23" H 8900 2200 60  0001 C CNN
-F 3 "" H 8900 2200 60  0000 C CNN
-	1    8900 2200
-	1    0    0    -1
-$EndComp
 Text Label 3550 6400 0    60   ~ 0
 PD1_IN
@@
 P 5700 4850
 F 0 "Q1" H 5700 4701 40  0000 R CNN
-F 1 "nMOS" H 5700 5000 40  0000 R CNN
-F 2 "SMD_Packages:SOT-23-GDS" H 5570 4952 29  0001 C CNN
-F 3 "" H 5700 4850 60  0000 C CNN
+F 1 "2N7002" H 5700 5000 40  0000 R CNN
+F 2 "SMD_Packages:SOT-23" H 5570 4952 29  0001 C CNN
+F 3 "http://www.nxp.com/documents/data_sheet/2N7002P.pdf" H 5700 4850 60  0001 C CNN
 	1    5700 4850
 	1    0    0    -1
@@
 F 3 "" H 7150 4900 60  0000 C CNN
 	1    7150 4900
-	1    0    0    -1
-$EndComp
-$Comp
-L DIODE D3
-U 1 1 546C4176
-P 8900 4550
-F 0 "D3" H 8900 4650 40  0000 C CNN
-F 1 "DIODE" H 8900 4450 40  0000 C CNN
-F 2 "SMD_Packages:SOT-23" H 8900 4550 60  0001 C CNN
-F 3 "" H 8900 4550 60  0000 C CNN
-	1    8900 4550
 	1    0    0    -1
 $EndComp
@@
 P 5750 2500
 F 0 "Q2" H 5750 2351 40  0000 R CNN
-F 1 "nMOS" H 5750 2650 40  0000 R CNN
-F 2 "SMD_Packages:SOT-23-GDS" H 5620 2602 29  0001 C CNN
-F 3 "" H 5750 2500 60  0000 C CNN
+F 1 "2N7002" H 5750 2650 40  0000 R CNN
+F 2 "SMD_Packages:SOT-23" H 5620 2602 29  0001 C CNN
+F 3 "http://www.nxp.com/documents/data_sheet/2N7002P.pdf" H 5750 2500 60  0001 C CNN
 	1    5750 2500
 	1    0    0    -1
@@
 Text Label 3550 3300 0    60   ~ 0
 3.3V_PROBE_0
+$Comp
+L SCHDPAK D1
+U 1 1 546E06E7
+P 8900 2250
+F 0 "D1" H 8900 2350 40  0000 C CNN
+F 1 "PMBD914,235" H 8900 2150 40  0000 C CNN
+F 2 "SMD_Packages:SOT-23" H 8900 2250 60  0001 C CNN
+F 3 "http://www.nxp.com/documents/data_sheet/PMBD914.pdf" H 8900 2250 60  0001 C CNN
+	1    8900 2250
+	1    0    0    -1
+$EndComp
+Wire Wire Line
+	9100 2250 9100 2200
+$Comp
+L SCHDPAK D3
+U 1 1 546E0977
+P 8900 4600
+F 0 "D3" H 8900 4700 40  0000 C CNN
+F 1 "PMBD914,235" H 8900 4500 40  0000 C CNN
+F 2 "SMD_Packages:SOT-23" H 8900 4600 60  0001 C CNN
+F 3 "http://www.nxp.com/documents/data_sheet/PMBD914.pdf" H 8900 4600 60  0001 C CNN
+	1    8900 4600
+	1    0    0    -1
+$EndComp
+Wire Wire Line
+	9100 4600 9100 4550
 $EndSCHEMATC

Commit message: first pass layout; one probe "done"
Parts:
- added C8: 100nF, parts:SMD-0402, symbol C
- added R8: 10kR, parts:SMD-0402, symbol R
Connections:
- wire segments 127 -> 130

Commit message: pinswap on PD diodes, second probe done. capacitances are approximate. ready to build, but next up is an experiment to maximize "edge" capacitance (at the expense of "substrate" capacitance).
Parts:
- removed D1, D3: PMBD914,235, SMD_Packages:SOT-23, symbol SCHDPAK
- added D1, D3: PMBD914,235, SMD_Packages:SOT-23, symbol DSOT23
Changed lines of the file:
@@
 LIBS:valves
 LIBS:parts
+LIBS:soil-moisture-module-cache
 EELAYER 24 0
 EELAYER END
@@
 ~RESET
 $Comp
-L +3.3V #PWR6
+L +3.3V #PWR01
 U 1 1 546BC650
 P 2800 1300
-F 0 "#PWR6" H 2800 1260 30  0001 C CNN
+F 0 "#PWR01" H 2800 1260 30  0001 C CNN
 F 1 "+3.3V" H 2800 1410 30  0000 C CNN
 F 2 "" H 2800 1300 60  0000 C CNN
@@
 $EndComp
 $Comp
-L GND #PWR5
+L GND #PWR02
 U 1 1 546BC69E
 P 2650 1400
-F 0 "#PWR5" H 2650 1400 30  0001 C CNN
+F 0 "#PWR02" H 2650 1400 30  0001 C CNN
 F 1 "GND" H 2650 1330 30  0001 C CNN
 F 2 "" H 2650 1400 60  0000 C CNN
@@
 $EndComp
 $Comp
-L +3.3V #PWR1
+L +3.3V #PWR03
 U 1 1 546BC8AA
 P 1250 6100
-F 0 "#PWR1" H 1250 6060 30  0001 C CNN
+F 0 "#PWR03" H 1250 6060 30  0001 C CNN
 F 1 "+3.3V" H 1250 6210 30  0000 C CNN
 F 2 "" H 1250 6100 60  0000 C CNN
@@
 $EndComp
 $Comp
-L GND #PWR2
+L GND #PWR04
 U 1 1 546BC8B0
 P 1250 7500
-F 0 "#PWR2" H 1250 7500 30  0001 C CNN
+F 0 "#PWR04" H 1250 7500 30  0001 C CNN
 F 1 "GND" H 1250 7430 30  0001 C CNN
 F 2 "" H 1250 7500 60  0000 C CNN
@@
 $EndComp
 $Comp
-L GND #PWR9
+L GND #PWR05
 U 1 1 546BF17D
 P 5200 7500
-F 0 "#PWR9" H 5200 7500 30  0001 C CNN
+F 0 "#PWR05" H 5200 7500 30  0001 C CNN
 F 1 "GND" H 5200 7430 30  0001 C CNN
 F 2 "" H 5200 7500 60  0000 C CNN
@@
 $EndComp
 $Comp
-L GND #PWR4
+L GND #PWR06
 U 1 1 546CC251
 P 2000 5250
-F 0 "#PWR4" H 2000 5250 30  0001 C CNN
+F 0 "#PWR06" H 2000 5250 30  0001 C CNN
 F 1 "GND" H 2000 5180 30  0001 C CNN
 F 2 "" H 2000 5250 60  0000 C CNN
@@
 GND1
 $Comp
-L +3.3V #PWR3
+L +3.3V #PWR07
 U 1 1 546CDDFD
 P 1900 3300
-F 0 "#PWR3" H 1900 3260 30  0001 C CNN
+F 0 "#PWR07" H 1900 3260 30  0001 C CNN
 F 1 "+3.3V" H 1900 3410 30  0000 C CNN
 F 2 "" H 1900 3300 60  0000 C CNN
@@
 3.3V_PROBE_0
 $Comp
-L SCHDPAK D1
-U 1 1 546E06E7
-P 8900 2250
-F 0 "D1" H 8900 2350 40  0000 C CNN
-F 1 "PMBD914,235" H 8900 2150 40  0000 C CNN
-F 2 "SMD_Packages:SOT-23" H 8900 2250 60  0001 C CNN
-F 3 "http://www.nxp.com/documents/data_sheet/PMBD914.pdf" H 8900 2250 60  0001 C CNN
-	1    8900 2250
-	1    0    0    -1
-$EndComp
-$Comp
-L SCHDPAK D3
-U 1 1 546E0977
-P 8900 4600
-F 0 "D3" H 8900 4700 40  0000 C CNN
-F 1 "PMBD914,235" H 8900 4500 40  0000 C CNN
-F 2 "SMD_Packages:SOT-23" H 8900 4600 60  0001 C CNN
-F 3 "http://www.nxp.com/documents/data_sheet/PMBD914.pdf" H 8900 4600 60  0001 C CNN
-	1    8900 4600
-	1    0    0    -1
-$EndComp
-$Comp
 L R R8
 U 1 1 546E7327
@@
 $EndComp
 $Comp
-L +3.3V #PWR7
+L +3.3V #PWR08
 U 1 1 546E732E
 P 3200 1600
-F 0 "#PWR7" H 3200 1560 30  0001 C CNN
+F 0 "#PWR08" H 3200 1560 30  0001 C CNN
 F 1 "+3.3V" H 3200 1710 30  0000 C CNN
 F 2 "" H 3200 1600 60  0000 C CNN
@@
 	3200 2800 3200 2900
 $Comp
-L GND #PWR8
+L GND #PWR09
 U 1 1 546E8823
 P 3200 2900
-F 0 "#PWR8" H 3200 2900 30  0001 C CNN
+F 0 "#PWR09" H 3200 2900 30  0001 C CNN
 F 1 "GND" H 3200 2830 30  0001 C CNN
 F 2 "" H 3200 2900 60  0000 C CNN
@@
 	1    0    0    -1
 $EndComp
+$Comp
+L DSOT23 D3
+U 1 1 546CFD3D
+P 8900 4600
+F 0 "D3" H 8900 4700 40  0000 C CNN
+F 1 "PMBD914,235" H 8900 4500 40  0000 C CNN
+F 2 "SMD_Packages:SOT-23" H 8900 4600 60  0001 C CNN
+F 3 "http://www.nxp.com/documents/data_sheet/PMBD914.pdf" H 8900 4600 60  0001 C CNN
+	1    8900 4600
+	1    0    0    -1
+$EndComp
+$Comp
+L DSOT23 D1
+U 1 1 546D0022
+P 8900 2250
+F 0 "D1" H 8900 2350 40  0000 C CNN
+F 1 "PMBD914,235" H 8900 2150 40  0000 C CNN
+F 2 "SMD_Packages:SOT-23" H 8900 2250 60  0001 C CNN
+F 3 "http://www.nxp.com/documents/data_sheet/PMBD914.pdf" H 8900 2250 60  0001 C CNN
+	1    8900 2250
+	1    0    0    -1
+$EndComp
